File: eagle/lb_single-sided_uno_v2.sch (EAGLE design)
At the start: 13 parts

Commit message: updated board designs and docs
Parts:
- PCB1: value ARDUINO_UNO -> ARDUINO_UNO_V2; device E14_Arduino_revC:ARDUINO_UNO -> E14_Arduino_revC:ARDUINO_UNO_V2
Changed lines of the file:
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@@
 </classes>
 <parts>
-<part name="PCB1" library="E14_Arduino_revC" deviceset="ARDUINO_UNO" device=""/>
+<part name="PCB1" library="E14_Arduino_revC" deviceset="ARDUINO_UNO_V2" device=""/>
 <part name="RED" library="fab" deviceset="LED" device="FAB1206" value="LEDFAB1206"/>
 <part name="GREEN" library="fab" deviceset="LED" device="FAB1206" value="LEDFAB1206"/>
