File: eagle/lb_uno_v1.3.sch (EAGLE design)
At the start: 16 parts, among them SW1 Button, SW3 Encoder

Commit message: updated board designs and docs
Parts:
- PCB1: value ARDUINO_UNO -> ARDUINO_UNO_V2; device E14_Arduino_revC:ARDUINO_UNO -> E14_Arduino_revC:ARDUINO_UNO_V2
- R1: value 330 -> 10k
- R4: value 10k -> 330
- SW3: value Encoder -> Rotary Encoder
Connections:
- net D10: now also R4.1; no longer R3.1
- net D7: now also R1.2; no longer R4.2
- net D8: now also R2.2; no longer R1.2
- net D9: now also R3.1; no longer R2.1
- net GND: now also R1.1; no longer R4.1
- net N$1: now also R2.1; no longer R1.1
- net N$2: now also R3.2; no longer R2.2
- net N$3: now also R4.2; no longer R3.2
Other:
- moved on the sheet: R1, R2, R3, R4
Changed lines of the file:
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@@
 <?xml version="1.0" encoding="utf-8"?>
 <!DOCTYPE eagle SYSTEM "eagle.dtd">
-<eagle version="9.1.1">
+<eagle version="9.6.2">
 <drawing>
 <settings>
@@
 </classes>
 <parts>
-<part name="PCB1" library="E14_Arduino_revC" deviceset="ARDUINO_UNO" device=""/>
+<part name="PCB1" library="E14_Arduino_revC" deviceset="ARDUINO_UNO_V2" device=""/>
 <part name="RED" library="fab" deviceset="LED" device="5MM" value="LED"/>
 <part name="SW1" library="adafruit" library_urn="urn:adsk.eagle:library:420" deviceset="SWITCH_PUSHBUTTON" device="EVQ-PE" package3d_urn="urn:adsk.eagle:package:6240957/1" value="Button"/>
-<part name="R1" library="adafruit" library_urn="urn:adsk.eagle:library:420" deviceset="R-US_" device="0207/9" package3d_urn="urn:adsk.eagle:package:6240935/1" value="330"/>
-<part name="R4" library="adafruit" library_urn="urn:adsk.eagle:library:420" deviceset="R-US_" device="0207/9" package3d_urn="urn:adsk.eagle:package:6240935/1" value="10k"/>
+<part name="R2" library="adafruit" library_urn="urn:adsk.eagle:library:420" deviceset="R-US_" device="0207/9" package3d_urn="urn:adsk.eagle:package:6240935/1" value="330"/>
+<part name="R1" library="adafruit" library_urn="urn:adsk.eagle:library:420" deviceset="R-US_" device="0207/9" package3d_urn="urn:adsk.eagle:package:6240935/1" value="10k"/>
 <part name="R6" library="pot" library_urn="urn:adsk.eagle:library:331" deviceset="TRIM_US-" device="B25P" package3d_urn="urn:adsk.eagle:package:22684/1" value="POT"/>
 <part name="GND6" library="supply1" library_urn="urn:adsk.eagle:library:371" deviceset="GND" device=""/>
 <part name="RGBLED" library="adafruit" library_urn="urn:adsk.eagle:library:420" deviceset="RGBLED_CA" device="-5MM" package3d_urn="urn:adsk.eagle:package:6240652/1" value="RGBLED"/>
-<part name="SW3" library="switch-alps" library_urn="urn:adsk.eagle:library:373" deviceset="EC12E_SW" device="" package3d_urn="urn:adsk.eagle:package:27083/1" value="Encoder"/>
+<part name="SW3" library="switch-alps" library_urn="urn:adsk.eagle:library:373" deviceset="EC12E_SW" device="" package3d_urn="urn:adsk.eagle:package:27083/1" value="Rotary Encoder"/>
 <part name="GND8" library="supply1" library_urn="urn:adsk.eagle:library:371" deviceset="GND" device=""/>
 <part name="R8" library="adafruit" library_urn="urn:adsk.eagle:library:420" deviceset="R-US_" device="0207/9" package3d_urn="urn:adsk.eagle:package:6240935/1" value="10k"/>
@@
 <part name="R9" library="adafruit" library_urn="urn:adsk.eagle:library:420" deviceset="R-US_" device="0207/9" package3d_urn="urn:adsk.eagle:package:6240935/1" value="10k"/>
 <part name="R10" library="adafruit" library_urn="urn:adsk.eagle:library:420" deviceset="R-US_" device="0207/9" package3d_urn="urn:adsk.eagle:package:6240935/1" value="10k"/>
-<part name="R2" library="adafruit" library_urn="urn:adsk.eagle:library:420" deviceset="R-US_" device="0207/9" package3d_urn="urn:adsk.eagle:package:6240935/1" value="330"/>
 <part name="R3" library="adafruit" library_urn="urn:adsk.eagle:library:420" deviceset="R-US_" device="0207/9" package3d_urn="urn:adsk.eagle:package:6240935/1" value="330"/>
+<part name="R4" library="adafruit" library_urn="urn:adsk.eagle:library:420" deviceset="R-US_" device="0207/9" package3d_urn="urn:adsk.eagle:package:6240935/1" value="330"/>
 <part name="R5" library="adafruit" library_urn="urn:adsk.eagle:library:420" deviceset="R-US_" device="0207/9" package3d_urn="urn:adsk.eagle:package:6240935/1" value="330"/>
 <part name="PH1" library="photo-elements" library_urn="urn:adsk.eagle:library:323" deviceset="A10" device="" package3d_urn="urn:adsk.eagle:package:22201/1" technology="60_12" value="Light"/>
@@
 <attribute name="VALUE" x="195.326" y="53.34" size="1.27" layer="96" rot="R90"/>
 </instance>
-<instance part="R1" gate="G$1" x="124.46" y="55.88" smashed="yes" rot="R90">
+<instance part="R2" gate="G$1" x="124.46" y="55.88" smashed="yes" rot="R90">
 <attribute name="NAME" x="122.9614" y="52.07" size="1.778" layer="95" rot="R90"/>
 <attribute name="VALUE" x="127.762" y="52.07" size="1.778" layer="96" rot="R90"/>
 </instance>
-<instance part="R4" gate="G$1" x="193.04" y="43.18" smashed="yes" rot="R90">
+<instance part="R1" gate="G$1" x="193.04" y="43.18" smashed="yes" rot="R90">
 <attribute name="NAME" x="191.5414" y="39.37" size="1.778" layer="95" rot="R90"/>
 <attribute name="VALUE" x="196.342" y="39.37" size="1.778" layer="96" rot="R90"/>
@@
 <instance part="SW3" gate="G$1" x="294.64" y="38.1" smashed="yes">
 <attribute name="PART" x="290.83" y="38.1" size="1.27" layer="95" rot="R90"/>
-<attribute name="VALUE" x="300.99" y="38.1" size="1.27" layer="96" rot="R90"/>
+<attribute name="VALUE" x="300.99" y="33.02" size="1.27" layer="96" rot="R90"/>
 </instance>
 <instance part="SW3" gate="G$2" x="309.88" y="53.34" smashed="yes" rot="R270">
@@
 <attribute name="VALUE" x="300.482" y="57.15" size="1.778" layer="96" rot="R90"/>
 </instance>
-<instance part="R2" gate="G$1" x="142.24" y="40.64" smashed="yes" rot="R90">
+<instance part="R3" gate="G$1" x="142.24" y="40.64" smashed="yes" rot="R90">
 <attribute name="NAME" x="140.7414" y="36.83" size="1.778" layer="95" rot="R90"/>
 <attribute name="VALUE" x="145.542" y="36.83" size="1.778" layer="96" rot="R90"/>
 </instance>
-<instance part="R3" gate="G$1" x="149.86" y="40.64" smashed="yes" rot="R90">
+<instance part="R4" gate="G$1" x="149.86" y="40.64" smashed="yes" rot="R90">
 <attribute name="NAME" x="148.3614" y="36.83" size="1.778" layer="95" rot="R90"/>
 <attribute name="VALUE" x="153.162" y="36.83" size="1.778" layer="96" rot="R90"/>
@@
 <net name="N$1" class="0">
 <segment>
-<pinref part="R1" gate="G$1" pin="1"/>
+<pinref part="R2" gate="G$1" pin="1"/>
 <pinref part="RED" gate="G$1" pin="A"/>
 <wire x1="124.46" y1="50.8" x2="124.46" y2="48.26" width="0.1524" layer="91"/>
@@
 </segment>
 <segment>
-<pinref part="R4" gate="G$1" pin="1"/>
+<pinref part="R1" gate="G$1" pin="1"/>
 <wire x1="193.04" y1="38.1" x2="193.04" y2="35.56" width="0.1524" layer="91"/>
 <pinref part="GND2" gate="1" pin="GND"/>
@@
 </segment>
 <segment>
-<pinref part="R3" gate="G$1" pin="1"/>
+<pinref part="R4" gate="G$1" pin="1"/>
 <wire x1="149.86" y1="35.56" x2="149.86" y2="33.02" width="0.1524" layer="91"/>
 <label x="149.86" y="33.02" size="1.27" layer="95" rot="R270" xref="yes"/>
@@
 </segment>
 <segment>
-<pinref part="R2" gate="G$1" pin="1"/>
+<pinref part="R3" gate="G$1" pin="1"/>
 <wire x1="142.24" y1="35.56" x2="142.24" y2="33.02" width="0.1524" layer="91"/>
 <label x="142.24" y="33.02" size="1.27" layer="95" rot="R270" xref="yes"/>
@@
 <pinref part="RGBLED" gate="G$1" pin="RED"/>
 <wire x1="144.78" y1="48.26" x2="144.78" y2="45.72" width="0.1524" layer="91"/>
-<pinref part="R2" gate="G$1" pin="2"/>
+<pinref part="R3" gate="G$1" pin="2"/>
 <wire x1="144.78" y1="45.72" x2="142.24" y2="45.72" width="0.1524" layer="91"/>
 </segment>
@@
 <segment>
 <pinref part="RGBLED" gate="G$1" pin="GREEN"/>
-<pinref part="R3" gate="G$1" pin="2"/>
+<pinref part="R4" gate="G$1" pin="2"/>
 <wire x1="149.86" y1="48.26" x2="149.86" y2="45.72" width="0.1524" layer="91"/>
 </segment>
@@
 </segment>
 <segment>
-<pinref part="R1" gate="G$1" pin="2"/>
+<pinref part="R2" gate="G$1" pin="2"/>
 <wire x1="124.46" y1="60.96" x2="124.46" y2="63.5" width="0.1524" layer="91"/>
 <label x="124.46" y="63.5" size="1.27" layer="95" rot="R90" xref="yes"/>
@@
 <segment>
 <pinref part="SW1" gate="G$1" pin="P$1"/>
-<pinref part="R4" gate="G$1" pin="2"/>
+<pinref part="R1" gate="G$1" pin="2"/>
 <wire x1="193.04" y1="50.8" x2="193.04" y2="48.26" width="0.1524" layer="91"/>
 <wire x1="193.04" y1="50.8" x2="195.58" y2="50.8" width="0.1524" layer="91"/>
